File: display_connector.sch (KiCad schematic (older format))
At the start: 1 part, among them J2 Display

Commit message: first version
Connections:
- net L4_1: now also J2.33 (P33); no longer J2.27 (P27)
- net L4_2: now also J2.32 (P32); no longer J2.28 (P28)
- net L4_3: now also J2.31 (P31); no longer J2.29 (P29)
- net L4_5: now also J2.29 (P29); no longer J2.31 (P31)
- net L4_6: now also J2.28 (P28); no longer J2.32 (P32)
- net L4_7: now also J2.27 (P27); no longer J2.33 (P33)
Changed lines of the file:
@@
 Wire Bus Line
 	2350 1150 2350 4950
-Text Label 2900 3350 0    60   ~ 0
+Text Label 2900 3950 0    60   ~ 0
 L4_1
-Text Label 2900 3450 0    60   ~ 0
+Text Label 2900 3850 0    60   ~ 0
 L4_2
-Text Label 2900 3550 0    60   ~ 0
+Text Label 2900 3750 0    60   ~ 0
 L4_3
 Text Label 2900 3650 0    60   ~ 0
 L4_4
-Text Label 2900 3750 0    60   ~ 0
+Text Label 2900 3550 0    60   ~ 0
 L4_5
-Text Label 2900 3850 0    60   ~ 0
+Text Label 2900 3450 0    60   ~ 0
 L4_6
-Text Label 2900 3950 0    60   ~ 0
+Text Label 2900 3350 0    60   ~ 0
 L4_7
 Text Label 2500 4050 0    60   ~ 0
