File: vfd_driver.sch (KiCad schematic (older format))
At the start: 36 parts, among them CON1 AVR-ISP-6, J1 PWR, J6 MH, J7 MH, J8 MH, J9 MH, U1 ATTINY2313-20SU, U10 74HC595, U11 74HC595, U12 74HC595, U13 74HC595, U14 ULN2803A, U15 ULN2803A, U16 ULN2003, U17 ULN2003, U18 LM1117-3.3, U2 74HC595, U3 74HC595, U4 74HC595, U5 74HC595, U6 ULN2803A, U7 ULN2003, U8 ULN2003, U9 ULN2003

Commit message: first version
Parts:
- removed D3, D4: LED, LEDs:LED_0805, symbol LED
- removed R6, R7: 470, Resistors_SMD:R_1206, symbol R_Small
- added R10, R11, R12, R13, R14, R15, R8, R9: 0, Resistors_SMD:R_1206, symbol R_Small
Connections:
- net G11: now also U6.11 (O8); no longer U6.18 (O1)
- net G12: now also U6.12 (O7); no longer U6.17 (O2)
- net G13: now also U6.13 (O6); no longer U6.16 (O3)
- net G14: now also U6.14 (O5); no longer U6.15 (O4)
- net G15: now also U6.15 (O4); no longer U6.14 (O5)
- net G16: now also U6.16 (O3); no longer U6.13 (O6)
- net G17: now also U6.17 (O2); no longer U6.12 (O7)
- net G18: now also U6.18 (O1); no longer U6.11 (O8)
- net G21: now also U14.11 (O8); no longer U14.18 (O1)
- net G22: now also U14.12 (O7); no longer U14.17 (O2)
- net G23: now also U14.13 (O6); no longer U14.16 (O3)
- net G24: now also U14.14 (O5); no longer U14.15 (O4)
- net G25: now also U14.15 (O4); no longer U14.14 (O5)
- net G26: now also U14.16 (O3); no longer U14.13 (O6)
- net G27: now also U14.17 (O2); no longer U14.12 (O7)
- net G28: now also U14.18 (O1); no longer U14.11 (O8)
- net G31: now also U15.11 (O8); no longer U15.18 (O1)
- net G32: now also U15.12 (O7); no longer U15.17 (O2)
- net G33: now also U15.13 (O6); no longer U15.16 (O3)
- net G34: now also U15.14 (O5); no longer U15.15 (O4)
- net G35: now also U15.15 (O4); no longer U15.14 (O5)
- net G36: now also U15.16 (O3); no longer U15.13 (O6)
- net G37: now also U15.17 (O2); no longer U15.12 (O7)
- net G38: now also U15.18 (O1); no longer U15.11 (O8)
- net L11: now also U7.10 (O7); no longer U7.16 (O1)
- net L12: now also U7.11 (O6); no longer U7.15 (O2)
- net L13: now also U7.12 (O5); no longer U7.14 (O3)
- net L15: now also U7.14 (O3); no longer U7.12 (O5)
- net L16: now also U7.15 (O2); no longer U7.11 (O6)
- net L17: now also U7.16 (O1); no longer U7.10 (O7)
- net L21: now also U8.10 (O7); no longer U8.16 (O1)
- net L22: now also U8.11 (O6); no longer U8.15 (O2)
- net L23: now also U8.12 (O5); no longer U8.14 (O3)
- net L25: now also U8.14 (O3); no longer U8.12 (O5)
- net L26: now also U8.15 (O2); no longer U8.11 (O6)
- net L27: now also U8.16 (O1); no longer U8.10 (O7)
- net L31: now also U16.10 (O7); no longer U16.16 (O1)
- net L32: now also U16.11 (O6); no longer U16.15 (O2)
- net L33: now also U16.12 (O5); no longer U16.14 (O3)
- net L35: now also U16.14 (O3); no longer U16.12 (O5)
- net L36: now also U16.15 (O2); no longer U16.11 (O6)
- net L37: now also U16.16 (O1); no longer U16.10 (O7)
- net L51: now also U17.10 (O7); no longer U17.16 (O1)
- net L52: now also U17.11 (O6); no longer U17.15 (O2)
- net L53: now also U17.12 (O5); no longer U17.14 (O3)
- net L55: now also U17.14 (O3); no longer U17.12 (O5)
- net L56: now also U17.15 (O2); no longer U17.11 (O6)
- net L57: now also U17.16 (O1); no longer U17.10 (O7)
- net RCLK_0: now also U1.4 (PA1(XTAL2)); no longer U1.12 ((PCINT0/AIN0)PB0)
- net RCLK_1: now also U1.3 ((TXD)PD1); no longer U1.6 ((CKOUT/XCK/INT0)PD2)
- net RCLK_2: now also U1.2 ((RXD)PD0); no longer U1.7 ((INT1)PD3)
- net RCLK_3: now also U1.9 ((OC0B/T1)PD5); no longer U1.8 ((T0)PD4)
- net RCLK_4: now also U1.8 ((T0)PD4); no longer U1.9 ((OC0B/T1)PD5)
- net RCLK_5: now also U1.7 ((INT1)PD3); no longer U1.11 ((ICP)PD6)
- net RCLK_6: now also U1.6 ((CKOUT/XCK/INT0)PD2); no longer U1.15 ((PCINT3/OC1A)PB3)
- net RCLK_7: now also U1.5 (PA0(XTAL1)); no longer U1.16 ((PCINT4/OC1B)PB4)
- net SER: now also U1.12 ((PCINT0/AIN0)PB0), R10.2, R11.2, R12.2, R13.2, R14.2, R15.2, R8.2, R9.2; no longer U1.13 ((PCINT1/AIN1)PB1), U10.14 (SER), U11.14 (SER), U12.14 (SER), U13.14 (SER), U2.14 (SER), U3.14 (SER), U4.14 (SER), U5.14 (SER)
- net SRCLK: now also U1.14 ((PCINT2/OC0A)PB2); no longer U1.2 ((RXD)PD0)
- net SRCLR: now also U1.13 ((PCINT1/AIN1)PB1); no longer U1.3 ((TXD)PD1)
- net at U13.1 (QB): now also U17.7 (I7); no longer U17.1 (I1)
- net at U13.2 (QC): now also U17.6 (I6); no longer U17.2 (I2)
- net at U13.3 (QD): now also U17.5 (I5); no longer U17.3 (I3)
- net at U13.5 (QF): now also U17.3 (I3); no longer U17.5 (I5)
- net at U13.6 (QG): now also U17.2 (I2); no longer U17.6 (I6)
- net at U13.7 (QH): now also U17.1 (I1); no longer U17.7 (I7)
- net at U5.1 (QB): now also U9.7 (I7); no longer U9.1 (I1)
- net at U5.2 (QC): now also U9.6 (I6); no longer U9.2 (I2)
- net at U5.3 (QD): now also U9.5 (I5); no longer U9.3 (I3)
- net at U5.5 (QF): now also U9.3 (I3); no longer U9.5 (I5)
- net at U5.6 (QG): now also U9.2 (I2); no longer U9.6 (I6)
- net at U5.7 (QH): now also U9.1 (I1); no longer U9.7 (I7)
- net at U12.1 (QB): now also U16.7 (I7); no longer U16.1 (I1)
- net at U12.2 (QC): now also U16.6 (I6); no longer U16.2 (I2)
- net at U12.3 (QD): now also U16.5 (I5); no longer U16.3 (I3)
- net at U12.5 (QF): now also U16.3 (I3); no longer U16.5 (I5)
- net at U12.6 (QG): now also U16.2 (I2); no longer U16.6 (I6)
- net at U12.7 (QH): now also U16.1 (I1); no longer U16.7 (I7)
- net at U4.1 (QB): now also U8.7 (I7); no longer U8.1 (I1)
- net at U4.2 (QC): now also U8.6 (I6); no longer U8.2 (I2)
- net at U4.3 (QD): now also U8.5 (I5); no longer U8.3 (I3)
- net at U4.5 (QF): now also U8.3 (I3); no longer U8.5 (I5)
- net at U4.6 (QG): now also U8.2 (I2); no longer U8.6 (I6)
- net at U4.7 (QH): now also U8.1 (I1); no longer U8.7 (I7)
- net at U3.1 (QB): now also U7.7 (I7); no longer U7.1 (I1)
- net at U3.2 (QC): now also U7.6 (I6); no longer U7.2 (I2)
- net at U3.3 (QD): now also U7.5 (I5); no longer U7.3 (I3)
- net at U3.5 (QF): now also U7.3 (I3); no longer U7.5 (I5)
- net at U3.6 (QG): now also U7.2 (I2); no longer U7.6 (I6)
- net at U3.7 (QH): now also U7.1 (I1); no longer U7.7 (I7)
- net at U2.1 (QB): now also U6.7 (I7); no longer U6.2 (I2)
- net at U2.15 (QA): now also U6.8 (I8); no longer U6.1 (I1)
- net at U2.2 (QC): now also U6.6 (I6); no longer U6.3 (I3)
- net at U2.3 (QD): now also U6.5 (I5); no longer U6.4 (I4)
- net at U2.4 (QE): now also U6.4 (I4); no longer U6.5 (I5)
- net at U2.5 (QF): now also U6.3 (I3); no longer U6.6 (I6)
- net at U2.6 (QG): now also U6.2 (I2); no longer U6.7 (I7)
- net at U2.7 (QH): now also U6.1 (I1); no longer U6.8 (I8)
- net at U10.1 (QB): now also U14.7 (I7); no longer U14.2 (I2)
- net at U10.15 (QA): now also U14.8 (I8); no longer U14.1 (I1)
- net at U10.2 (QC): now also U14.6 (I6); no longer U14.3 (I3)
- net at U10.3 (QD): now also U14.5 (I5); no longer U14.4 (I4)
- net at U10.4 (QE): now also U14.4 (I4); no longer U14.5 (I5)
- net at U10.5 (QF): now also U14.3 (I3); no longer U14.6 (I6)
- net at U10.6 (QG): now also U14.2 (I2); no longer U14.7 (I7)
- net at U10.7 (QH): now also U14.1 (I1); no longer U14.8 (I8)
- net at U11.1 (QB): now also U15.7 (I7); no longer U15.2 (I2)
- net at U11.15 (QA): now also U15.8 (I8); no longer U15.1 (I1)
- net at U11.2 (QC): now also U15.6 (I6); no longer U15.3 (I3)
- net at U11.3 (QD): now also U15.5 (I5); no longer U15.4 (I4)
- net at U11.4 (QE): now also U15.4 (I4); no longer U15.5 (I5)
- net at U11.5 (QF): now also U15.3 (I3); no longer U15.6 (I6)
- net at U11.6 (QG): now also U15.2 (I2); no longer U15.7 (I7)
- net at U11.7 (QH): now also U15.1 (I1); no longer U15.8 (I8)
- new net: R15.1, U13.14 (SER)
- new net: R11.1, U5.14 (SER)
- new net: R14.1, U12.14 (SER)
- new net: R10.1, U4.14 (SER)
- new net: R9.1, U3.14 (SER)
- new net: R8.1, U2.14 (SER)
- new net: R12.1, U10.14 (SER)
- new net: R13.1, U11.14 (SER)
- no-connect marks 16 -> 13
Other:
- moved on the sheet: C1, D2, R1, R5, U14, U15, U16, U17, U6, U7, U8, U9
